File: MiniDiv/MiniDiv.kicad_sch (KiCad schematic)
At the start: 24 parts, among them Q1 2N3904, U1 L7805, U2 CD4040, U3 40106

Commit message: Updated schematics
Parts:
- added U4: 40106, symbol 4xxx:40106
- renumbered DIV_OUT_1 to CLOCK_OUT1, RESET_SW to RESET_SW1
Connections:
- net +5V: now also U4.14 (VDD)
- net Earth: now also U4.11, U4.13, U4.9
- net GND: now also U4.7 (VSS)
- net at U2.13 (Q7): now also U4.5
- net at U2.2 (Q5): now also U4.1
- net at U2.4 (Q6): now also U4.3
- new net OUT_128: U4.4
- new net OUT_256: U4.6
- new net OUT_64: U4.2
- no-connect marks 2 -> 5
Other:
- note added: "Clock Divider Core"
- note added: "Internal Clock"
- note added: "Inverters"
- note added: "Power"
- company: (none) -> benjiaomodular
- title: (none) -> MiniDiv
- moved on the sheet: C1, C2, C5, C6, CLOCK_IN1, CLOCK_OUT1, D1, D2, DIV_OUT_2, Q1, R1, R2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
