File: hardware/old_versions/MiniDiv v0.1/Eurorack Power.kicad_sch (KiCad schematic)
At the start: 3 parts, among them J1 IDC_2x05

Commit message: reorganized, updated license, finalized 0.2 circuit
Parts:
- C3, C4: Manufacturers Name YAGEO -> Murata Electronics; Manufacturers Part Number CC0805KRX7R9BB104 -> GRM21BR61E226ME44L
Changed lines of the file:
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@@
       (effects (font (size 1.27 1.27)) hide)
     )
-    (property "Manufacturers Part Number" "CC0805KRX7R9BB104" (id 6) (at 41.656 41.656 0)
+    (property "Manufacturers Part Number" "GRM21BR61E226ME44L" (id 6) (at 41.656 41.656 0)
       (effects (font (size 1.27 1.27)) hide)
     )
-    (property "Manufacturers Name" "YAGEO" (id 7) (at 41.656 41.656 0)
+    (property "Manufacturers Name" "Murata Electronics " (id 7) (at 41.656 41.656 0)
       (effects (font (size 1.27 1.27)) hide)
     )
@@
       (effects (font (size 1.27 1.27)) hide)
     )
-    (property "Manufacturers Part Number" "CC0805KRX7R9BB104" (id 6) (at 41.656 31.496 0)
+    (property "Manufacturers Part Number" "GRM21BR61E226ME44L" (id 6) (at 41.656 31.496 0)
       (effects (font (size 1.27 1.27)) hide)
     )
-    (property "Manufacturers Name" "YAGEO" (id 7) (at 41.656 31.496 0)
+    (property "Manufacturers Name" "Murata Electronics " (id 7) (at 41.656 31.496 0)
       (effects (font (size 1.27 1.27)) hide)
     )
