File: hardware/old_versions/MiniDiv v0.1/MiniDiv.kicad_sch (KiCad schematic)
At the start: 25 parts, among them Q1 2N3904, U1 L7805, U2 CD4040, U3 40106, U4 40106

Commit message: reorganized, updated license, finalized 0.2 circuit
Parts:
- added Q?: 2N3904, Package_TO_SOT_THT:TO-92_Inline, symbol Transistor_BJT:2N3904
- added R? (x2): 10k, Resistor_SMD:R_0603_1608Metric_Pad0.98x0.95mm_HandSolder, symbol Device:R
- added R?: 100k, Resistor_SMD:R_0603_1608Metric_Pad0.98x0.95mm_HandSolder, symbol Device:R
- added RESET_IN?: PJ-3001F, symbol Connector:AudioJack2_SwitchT
- C6: Manufacturers Name (none) -> Taiyo Yuden; Manufacturers Part Number (none) -> TMK212BBJ106KG8T
- D1, D2: footprint (none) -> LED_THT:LED_D3.0mm; Manufacturers Name (none) -> KENTO; Manufacturers Part Number (none) -> 3ARG4HWC
- R1, R2, R3, R4, R5, R6, R7, R8, R9: footprint (none) -> Resistor_SMD:R_0603_1608Metric_Pad0.98x0.95mm_HandSolder
Connections:
- net +5V: now also R?.2
- net Earth: now also Q?.1 (E), R?.1, RESET_IN?.S
- net INT_CLOCK: now also RESET_IN?.TN
- new net: Q?.2 (B), R?.2, R?.2
- new net: Q?.3 (C), R?.1
- new net: R?.1, RESET_IN?.T
