File: hardware/circuit/MiniDiv/Outputs.kicad_sch (KiCad schematic)
At the start: 32 parts

Commit message: v0.2 PCB
Parts:
- added D13, D14: LED, LED_SMD:LED_0805_2012Metric, symbol Device:LED
- added OUT_10, OUT_9: PJ3001F, benjiaomodular:AudioJack_3.5mm, symbol benjiaomodular:PJ3001F
- added R26, R27: 4.7k, Resistor_SMD:R_0603_1608Metric_Pad0.98x0.95mm_HandSolder, symbol Device:R
- added R28, R29: 1k, Resistor_SMD:R_0603_1608Metric_Pad0.98x0.95mm_HandSolder, symbol Device:R
- D10: renamed from D11; footprint LED_THT:LED_D3.0mm -> LED_SMD:LED_0805_2012Metric
- D11: renamed from D12; footprint LED_THT:LED_D3.0mm -> LED_SMD:LED_0805_2012Metric
- D12: renamed from D13; footprint LED_THT:LED_D3.0mm -> LED_SMD:LED_0805_2012Metric
- D5: renamed from D6; footprint LED_THT:LED_D3.0mm -> LED_SMD:LED_0805_2012Metric
- D6: renamed from D7; footprint LED_THT:LED_D3.0mm -> LED_SMD:LED_0805_2012Metric
- D7: renamed from D8; footprint LED_THT:LED_D3.0mm -> LED_SMD:LED_0805_2012Metric
- D8: renamed from D9; footprint LED_THT:LED_D3.0mm -> LED_SMD:LED_0805_2012Metric
- D9: renamed from D10; footprint LED_THT:LED_D3.0mm -> LED_SMD:LED_0805_2012Metric
- renumbered DIV_OUT1 to OUT_1, DIV_OUT2 to OUT_2, DIV_OUT3 to OUT_3, DIV_OUT4 to OUT_4, DIV_OUT5 to OUT_5, DIV_OUT6 to OUT_6, DIV_OUT7 to OUT_7, DIV_OUT8 to OUT_8, R11 to R10, R12 to R11, R13 to R12, R14 to R13, R15 to R14, R17 to R15, R18 to R16, R16 to R17, R19 to R18, R20 to R19, R21 to R20, R22 to R21, R23 to R22, R24 to R23, R25 to R24, R26 to R25
Connections:
- net GND: now also D13.1 (K), D14.1 (K), OUT_10.S, OUT_9.S
- new net: D14.2 (A), R27.2
- new net: D13.2 (A), R26.2
- new net: OUT_9.T, R28.1
- new net: OUT_10.T, R29.1
- new net OUT_1024: R27.1, R29.2
- new net OUT_512: R26.1, R28.2
- no-connect marks 8 -> 10

Commit message: Updated PCBs
Parts:
- D10, D11, D12, D13, D14, D5, D6, D7, D8, D9: URL (none) -> https://www.taydaelectronics.com/led-3mm-orange.html
- R14, R15, R16, R17, R22, R23, R24, R25, R28, R29: URL (none) -> https://mou.sr/3MKtPCB

Commit message: Added drawings and photos
Parts:
- D10, D11, D12, D13, D14, D5, D6, D7, D8, D9: Manufacturer (none) -> KENTO; Manufacturers Name KENTO -> (none); Manufacturers Part Number 3ARG4HWC -> (none); Part # (none) -> 3ARG4HWC
- OUT_1, OUT_10, OUT_2, OUT_3, OUT_4, OUT_5, OUT_6, OUT_7, OUT_8, OUT_9: Manufacturer (none) -> Tayda Electronics; Part # (none) -> PJ-3001F; URL (none) -> https://www.taydaelectronics.com/pj-3001f-3-5-mm-mono-phone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
- R10, R11, R12, R13, R18, R19, R20, R21, R26, R27: Manufacturer (none) -> YAGEO; Part # (none) -> RC0603FR-074K7L; URL (none) -> https://mou.sr/3Zl09mQ
- R14, R15, R16, R17, R22, R23, R24, R25, R28, R29: Manufacturer (none) -> YAGEO; Part # (none) -> RC0603FR-071KL
